File: CurrentControl.sch (KiCad schematic (older format))
At the start: 7 parts

Commit message: Initial Annotation
Parts:
- gave numbers to parts that had none: 7
Connections:
- net at Q301.3 (S), R303.1: now also U201.6 (-); no longer U201.2 (-)
- net at R301.1, RV301.3: now also U201.5 (+); no longer U201.3 (+)
- net at R302.2: now also U201.7; no longer U201.1
Changed lines of the file:
@@
 $EndDescr
 $Comp
-L Q_NMOS_DGS Q?
+L Q_NMOS_DGS Q301
 U 1 1 5B20DECB
 P 8600 3250
-F 0 "Q?" H 8550 3450 50  0000 L CNN
+F 0 "Q301" H 8550 3450 50  0000 L CNN
 F 1 "BUK9575" H 8300 3100 50  0000 L CNN
 F 2 "" H 8800 3350 50  0001 C CNN
@@
 $EndComp
 $Comp
-L R R?
+L R R303
 U 1 1 5B20DED3
 P 8700 4600
-F 0 "R?" V 8780 4600 50  0000 C CNN
+F 0 "R303" V 8780 4600 50  0000 C CNN
 F 1 "0.1" V 8700 4600 50  0000 C CNN
 F 2 "" V 8630 4600 50  0001 C CNN
@@
 $EndComp
 $Comp
-L R R?
+L R R301
 U 1 1 5B20DEE0
 P 4000 4500
-F 0 "R?" V 4080 4500 50  0000 C CNN
+F 0 "R301" V 4080 4500 50  0000 C CNN
 F 1 "R" V 4000 4500 50  0000 C CNN
 F 2 "" V 3930 4500 50  0001 C CNN
@@
 $EndComp
 $Comp
-L LMV358 U?
-U 1 1 5B20DEE7
+L LMV358 U201
+U 2 1 5B20DEE7
 P 5400 3250
-F 0 "U?" H 5400 3450 50  0000 L CNN
+F 0 "U201" H 5400 3450 50  0000 L CNN
 F 1 "LMV358" H 5400 3050 50  0000 L CNN
 F 2 "" H 5400 3250 50  0001 C CNN
 F 3 "" H 5400 3250 50  0001 C CNN
-	1    5400 3250
+	2    5400 3250
 	1    0    0    -1
 $EndComp
 $Comp
-L GND #PWR?
+L GND #PWR302
 U 1 1 5B20DEEE
 P 5300 3700
-F 0 "#PWR?" H 5300 3450 50  0001 C CNN
+F 0 "#PWR302" H 5300 3450 50  0001 C CNN
 F 1 "GND" H 5300 3550 50  0000 C CNN
 F 2 "" H 5300 3700 50  0001 C CNN
@@
 $EndComp
 $Comp
-L POT RV?
+L POT RV301
 U 1 1 5B20DEF4
 P 4000 3850
-F 0 "RV?" V 3825 3850 50  0000 C CNN
+F 0 "RV301" V 3825 3850 50  0000 C CNN
 F 1 "POT" V 3900 3850 50  0000 C CNN
 F 2 "" H 4000 3850 50  0001 C CNN
@@
 $EndComp
 $Comp
-L GND #PWR?
+L GND #PWR301
 U 1 1 5B20DEFB
 P 4750 2900
-F 0 "#PWR?" H 4750 2650 50  0001 C CNN
+F 0 "#PWR301" H 4750 2650 50  0001 C CNN
 F 1 "GND" H 4750 2750 50  0000 C CNN
 F 2 "" H 4750 2900 50  0001 C CNN
@@
 	4750 2800 4750 2900
 $Comp
-L C C?
+L C C301
 U 1 1 5B20DF16
 P 4750 2650
-F 0 "C?" H 4775 2750 50  0000 L CNN
+F 0 "C301" H 4775 2750 50  0000 L CNN
 F 1 "C" H 4775 2550 50  0000 L CNN
 F 2 "" H 4788 2500 50  0001 C CNN
@@
 	8900 1300 8700 1300
 $Comp
-L R R?
+L R R302
 U 1 1 5B20E5D2
 P 6350 3250
-F 0 "R?" V 6430 3250 50  0000 C CNN
+F 0 "R302" V 6430 3250 50  0000 C CNN
 F 1 "1K" V 6350 3250 50  0000 C CNN
 F 2 "" V 6280 3250 50  0001 C CNN

Commit message: Added footprints. Created initial netlist.
Parts:
- C301: footprint (none) -> Capacitors_SMD:C_0805_HandSoldering
- Q301: footprint (none) -> TO_SOT_Packages_THT:TO-220-3_Vertical
- R301, R302: footprint (none) -> Resistors_SMD:R_0805
- R303: footprint (none) -> Resistors_THT:R_Axial_DIN0516_L15.5mm_D5.0mm_P25.40mm_Horizontal
- RV301: footprint (none) -> Potentiometers:Potentiometer_WirePads_largePads
- U201: footprint (none) -> SMD_Packages:SOIC-8-N
Changed lines of the file:
@@
 F 0 "Q301" H 8550 3450 50  0000 L CNN
 F 1 "BUK9575" H 8300 3100 50  0000 L CNN
-F 2 "" H 8800 3350 50  0001 C CNN
+F 2 "TO_SOT_Packages_THT:TO-220-3_Vertical" H 8800 3350 50  0001 C CNN
 F 3 "" H 8600 3250 50  0001 C CNN
 F 4 "BUK9575-100A,127" H 8600 3250 60  0001 C CNN "MPN"
@@
 F 0 "R303" V 8780 4600 50  0000 C CNN
 F 1 "0.1" V 8700 4600 50  0000 C CNN
-F 2 "" V 8630 4600 50  0001 C CNN
+F 2 "Resistors_THT:R_Axial_DIN0516_L15.5mm_D5.0mm_P25.40mm_Horizontal" V 8630 4600 50  0001 C CNN
 F 3 "" H 8700 4600 50  0001 C CNN
 F 4 "AC01000001007JA100" V 8700 4600 60  0001 C CNN "MPN"
@@
 F 0 "R301" V 4080 4500 50  0000 C CNN
 F 1 "R" V 4000 4500 50  0000 C CNN
-F 2 "" V 3930 4500 50  0001 C CNN
+F 2 "Resistors_SMD:R_0805" V 3930 4500 50  0001 C CNN
 F 3 "" H 4000 4500 50  0001 C CNN
 	1    4000 4500
@@
 F 0 "U201" H 5400 3450 50  0000 L CNN
 F 1 "LMV358" H 5400 3050 50  0000 L CNN
-F 2 "" H 5400 3250 50  0001 C CNN
+F 2 "SMD_Packages:SOIC-8-N" H 5400 3250 50  0001 C CNN
 F 3 "" H 5400 3250 50  0001 C CNN
 	2    5400 3250
@@
 $EndComp
 $Comp
-L GND #PWR302
+L GND #PWR05
 U 1 1 5B20DEEE
 P 5300 3700
-F 0 "#PWR302" H 5300 3450 50  0001 C CNN
+F 0 "#PWR05" H 5300 3450 50  0001 C CNN
 F 1 "GND" H 5300 3550 50  0000 C CNN
 F 2 "" H 5300 3700 50  0001 C CNN
@@
 F 0 "RV301" V 3825 3850 50  0000 C CNN
 F 1 "POT" V 3900 3850 50  0000 C CNN
-F 2 "" H 4000 3850 50  0001 C CNN
+F 2 "Potentiometers:Potentiometer_WirePads_largePads" H 4000 3850 50  0001 C CNN
 F 3 "" H 4000 3850 50  0001 C CNN
 	1    4000 3850
@@
 $EndComp
 $Comp
-L GND #PWR301
+L GND #PWR06
 U 1 1 5B20DEFB
 P 4750 2900
-F 0 "#PWR301" H 4750 2650 50  0001 C CNN
+F 0 "#PWR06" H 4750 2650 50  0001 C CNN
 F 1 "GND" H 4750 2750 50  0000 C CNN
 F 2 "" H 4750 2900 50  0001 C CNN
@@
 F 0 "C301" H 4775 2750 50  0000 L CNN
 F 1 "C" H 4775 2550 50  0000 L CNN
-F 2 "" H 4788 2500 50  0001 C CNN
+F 2 "Capacitors_SMD:C_0805_HandSoldering" H 4788 2500 50  0001 C CNN
 F 3 "" H 4750 2650 50  0001 C CNN
 	1    4750 2650
@@
 F 0 "R302" V 6430 3250 50  0000 C CNN
 F 1 "1K" V 6350 3250 50  0000 C CNN
-F 2 "" V 6280 3250 50  0001 C CNN
+F 2 "Resistors_SMD:R_0805" V 6280 3250 50  0001 C CNN
 F 3 "" H 6350 3250 50  0001 C CNN
 	1    6350 3250

Commit message: Update connector footprints
Parts:
- added J1: Conn_01x01, Current:FA-T220-38E, symbol Conn_01x01
Changed lines of the file:
@@
 Text HLabel 9200 5300 2    60   Input ~ 0
 Current_Sink-
+$Comp
+L Conn_01x01 J1
+U 1 1 5B2868CB
+P 9950 3250
+F 0 "J1" H 9950 3350 50  0000 C CNN
+F 1 "Conn_01x01" H 9950 3150 50  0000 C CNN
+F 2 "Current:FA-T220-38E" H 9950 3250 50  0001 C CNN
+F 3 "" H 9950 3250 50  0001 C CNN
+	1    9950 3250
+	1    0    0    -1
+$EndComp
 $EndSCHEMATC

Commit message: Fixed divider resistors and found valus. Added pot footprint.
Parts:
- R301: value R -> 68K
- RV301: value POT -> 10K; footprint Potentiometers:Potentiometer_WirePads_largePads -> Current:P090L-02F25BR10K
Connections:
- wire segments 26 -> 24
Other:
- moved on the sheet: C301, R301, RV301
Changed lines of the file:
@@
 L R R301
 U 1 1 5B20DEE0
-P 4000 4500
-F 0 "R301" V 4080 4500 50  0000 C CNN
-F 1 "R" V 4000 4500 50  0000 C CNN
-F 2 "Resistors_SMD:R_0805" V 3930 4500 50  0001 C CNN
-F 3 "" H 4000 4500 50  0001 C CNN
-	1    4000 4500
+P 4200 4000
+F 0 "R301" V 4280 4000 50  0000 C CNN
+F 1 "68K" V 4200 4000 50  0000 C CNN
+F 2 "Resistors_SMD:R_0805" V 4130 4000 50  0001 C CNN
+F 3 "" H 4200 4000 50  0001 C CNN
+	1    4200 4000
 	1    0    0    -1
 $EndComp
@@
 L POT RV301
 U 1 1 5B20DEF4
-P 4000 3850
-F 0 "RV301" V 3825 3850 50  0000 C CNN
-F 1 "POT" V 3900 3850 50  0000 C CNN
-F 2 "Potentiometers:Potentiometer_WirePads_largePads" H 4000 3850 50  0001 C CNN
-F 3 "" H 4000 3850 50  0001 C CNN
-	1    4000 3850
+P 4200 4430
+F 0 "RV301" V 4025 4430 50  0000 C CNN
+F 1 "10K" V 4100 4430 50  0000 C CNN
+F 2 "Current:P090L-02F25BR10K" H 4200 4430 50  0001 C CNN
+F 3 "" H 4200 4430 50  0001 C CNN
+	1    4200 4430
 	1    0    0    -1
 $EndComp
@@
 L GND #PWR06
 U 1 1 5B20DEFB
-P 4750 2900
-F 0 "#PWR06" H 4750 2650 50  0001 C CNN
-F 1 "GND" H 4750 2750 50  0000 C CNN
-F 2 "" H 4750 2900 50  0001 C CNN
-F 3 "" H 4750 2900 50  0001 C CNN
-	1    4750 2900
+P 4750 2392
+F 0 "#PWR06" H 4750 2142 50  0001 C CNN
+F 1 "GND" H 4750 2242 50  0000 C CNN
+F 2 "" H 4750 2392 50  0001 C CNN
+F 3 "" H 4750 2392 50  0001 C CNN
+	1    4750 2392
 	1    0    0    -1
 $EndComp
-Wire Wire Line
-	8700 3450 8700 4450
-Wire Wire Line
-	5100 3350 4850 3350
-Wire Wire Line
-	4850 3350 4850 4100
-Wire Wire Line
-	4850 4100 8700 4100
-Connection ~ 8700 4100
-Wire Wire Line
-	4000 4000 4000 4350
-Wire Wire Line
-	4000 4650 4000 4900
-Wire Wire Line
-	4000 4900 8700 4900
-Connection ~ 8700 4900
-Wire Wire Line
-	5300 3550 5300 3700
-Wire Wire Line
-	4200 3850 4150 3850
-Wire Wire Line
-	5300 2400 5300 2950
-Wire Wire Line
-	4200 2400 5300 2400
-Wire Wire Line
-	8700 1300 8700 3050
-Wire Wire Line
-	4750 2800 4750 2900
 $Comp
 L C C301
 U 1 1 5B20DF16
-P 4750 2650
-F 0 "C301" H 4775 2750 50  0000 L CNN
-F 1 "C" H 4775 2550 50  0000 L CNN
-F 2 "Capacitors_SMD:C_0805_HandSoldering" H 4788 2500 50  0001 C CNN
-F 3 "" H 4750 2650 50  0001 C CNN
-	1    4750 2650
+P 4750 2142
+F 0 "C301" H 4775 2242 50  0000 L CNN
+F 1 "C" H 4775 2042 50  0000 L CNN
+F 2 "Capacitors_SMD:C_0805_HandSoldering" H 4788 1992 50  0001 C CNN
+F 3 "" H 4750 2142 50  0001 C CNN
+	1    4750 2142
 	1    0    0    -1
 $EndComp
-Connection ~ 4750 2400
-Connection ~ 4200 2400
-Wire Wire Line
-	4750 2500 4750 2400
-Connection ~ 4000 4150
-Wire Wire Line
-	4450 3150 5100 3150
-Wire Wire Line
-	4450 4150 4000 4150
-Wire Wire Line
-	4450 3150 4450 4150
 Text GLabel 3250 1850 0    60   Input ~ 0
 2.7V
-Wire Wire Line
-	3250 1850 4200 1850
-Connection ~ 4200 1850
-Wire Wire Line
-	4200 1850 4200 3850
 Text HLabel 8900 1300 2    60   Input ~ 0
 Current_Sink+
-Wire Wire Line
-	8900 1300 8700 1300
 $Comp
 L R R302
@@
 	0    1    1    0
 $EndComp
-Wire Wire Line
-	6200 3250 5700 3250
-Wire Wire Line
-	6500 3250 8400 3250
-Wire Wire Line
-	7500 3250 7500 950
-Wire Wire Line
-	7500 950  8900 950
-Connection ~ 7500 3250
 Text HLabel 8900 950  2    60   Input ~ 0
 FET_Gate
-Wire Wire Line
-	8700 4750 8700 5300
-Wire Wire Line
-	8700 5300 9200 5300
 Text HLabel 9200 5300 2    60   Input ~ 0
 Current_Sink-
@@
 	1    0    0    -1
 $EndComp
+Wire Wire Line
+	8700 3450 8700 4450
+Wire Wire Line
+	5100 3350 4850 3350
+Wire Wire Line
+	4850 3350 4850 4100
+Wire Wire Line
+	4850 4100 8700 4100
+Connection ~ 8700 4100
+Connection ~ 8700 4900
+Wire Wire Line
+	5300 3550 5300 3700
+Wire Wire Line
+	8700 1300 8700 3050
+Wire Wire Line
+	4750 2292 4750 2392
+Wire Wire Line
+	4450 3150 5100 3150
+Wire Wire Line
+	3250 1850 5300 1850
+Connection ~ 4200 1850
+Wire Wire Line
+	4200 1850 4200 3850
+Wire Wire Line
+	8900 1300 8700 1300
+Wire Wire Line
+	6200 3250 5700 3250
+Wire Wire Line
+	6500 3250 8400 3250
+Wire Wire Line
+	7500 3250 7500 950
+Wire Wire Line
+	7500 950  8900 950
+Connection ~ 7500 3250
+Wire Wire Line
+	8700 4750 8700 5300
+Wire Wire Line
+	8700 5300 9200 5300
+Wire Wire Line
+	5300 1850 5300 2950
+Wire Wire Line
+	4750 1990 4750 1850
+Connection ~ 4750 1850
+Wire Wire Line
+	4450 3150 4450 4200
+Wire Wire Line
+	4450 4200 4200 4200
+Wire Wire Line
+	4200 4150 4200 4280
+Wire Wire Line
+	4350 4900 8700 4900
+Wire Wire Line
+	4350 4900 4350 4430
+Connection ~ 4200 4200
 $EndSCHEMATC
