File: CurrentSinkorSwim.sch (KiCad schematic (older format))
At the start: 10 parts

Commit message: adding new sheets and voltage control circuit
Parts:
- removed C? (x2): C, symbol C
- removed Q?: Q_NMOS_DGS, symbol Q_NMOS_DGS
- removed R? (x2): R, symbol R
- removed RV?: POT, symbol POT
- removed U? (x2): LMV358, symbol LMV358
- removed U?: TC1016, TO_SOT_Packages_THT:TO-220_Vertical, symbol TC1016
- added J?: Conn_01x03, symbol Conn_01x03
- added J?: Conn_01x02, symbol Conn_01x02
Connections:
- wire segments 27 -> 18
Other:
- note added: "Battery Pack"
- note added: "Current Sink Input"
- moved on the sheet: J?

Commit message: Initial Annotation
Parts:
- gave numbers to parts that had none: 3
Changed lines of the file:
@@
 $EndDescr
 $Comp
-L Conn_01x02 J?
+L Conn_01x02 J103
 U 1 1 5B1871C6
 P 7350 2250
-F 0 "J?" H 7350 2350 50  0000 C CNN
+F 0 "J103" H 7350 2350 50  0000 C CNN
 F 1 "Conn_01x02" V 7450 2200 50  0000 C CNN
 F 2 "" H 7350 2250 50  0001 C CNN
@@
 	6050 1950 6050 2900
 $Comp
-L Conn_01x03 J?
+L Conn_01x03 J102
 U 1 1 5B1CFFCF
 P 6050 1750
-F 0 "J?" H 6050 1950 50  0000 C CNN
+F 0 "J102" H 6050 1950 50  0000 C CNN
 F 1 "Conn_01x03" V 6150 1750 50  0000 C CNN
 F 2 "" H 6050 1750 50  0001 C CNN
@@
 	5950 2000 5950 1950
 $Comp
-L Conn_01x02 J?
+L Conn_01x02 J101
 U 1 1 5B1D04AE
 P 3000 2100
-F 0 "J?" H 3000 2200 50  0000 C CNN
+F 0 "J101" H 3000 2200 50  0000 C CNN
 F 1 "Conn_01x02" V 3100 2050 50  0000 C CNN
 F 2 "" H 3000 2100 50  0001 C CNN
@@
 $EndComp
 $Comp
-L GND #PWR?
+L GND #PWR101
 U 1 1 5B1D0556
 P 3350 2550
-F 0 "#PWR?" H 3350 2300 50  0001 C CNN
+F 0 "#PWR101" H 3350 2300 50  0001 C CNN
 F 1 "GND" H 3350 2400 50  0000 C CNN
 F 2 "" H 3350 2550 50  0001 C CNN
@@
 	4800 4650 4500 4650
 $Comp
-L GND #PWR?
+L GND #PWR102
 U 1 1 5B2120C5
 P 7000 6300
-F 0 "#PWR?" H 7000 6050 50  0001 C CNN
+F 0 "#PWR102" H 7000 6050 50  0001 C CNN
 F 1 "GND" H 7000 6150 50  0000 C CNN
 F 2 "" H 7000 6300 50  0001 C CNN

Commit message: Added footprints. Created initial netlist.
Parts:
- J101, J103: footprint (none) -> Pin_Headers:Pin_Header_Angled_1x02_Pitch2.54mm
- J102: footprint (none) -> Pin_Headers:Pin_Header_Angled_1x03_Pitch2.54mm
Changed lines of the file:
@@
 F 0 "J103" H 7350 2350 50  0000 C CNN
 F 1 "Conn_01x02" V 7450 2200 50  0000 C CNN
-F 2 "" H 7350 2250 50  0001 C CNN
+F 2 "Pin_Headers:Pin_Header_Angled_1x02_Pitch2.54mm" H 7350 2250 50  0001 C CNN
 F 3 "" H 7350 2250 50  0001 C CNN
 	1    7350 2250
@@
 F 0 "J102" H 6050 1950 50  0000 C CNN
 F 1 "Conn_01x03" V 6150 1750 50  0000 C CNN
-F 2 "" H 6050 1750 50  0001 C CNN
+F 2 "Pin_Headers:Pin_Header_Angled_1x03_Pitch2.54mm" H 6050 1750 50  0001 C CNN
 F 3 "" H 6050 1750 50  0001 C CNN
 	1    6050 1750
@@
 F 0 "J101" H 3000 2200 50  0000 C CNN
 F 1 "Conn_01x02" V 3100 2050 50  0000 C CNN
-F 2 "" H 3000 2100 50  0001 C CNN
+F 2 "Pin_Headers:Pin_Header_Angled_1x02_Pitch2.54mm" H 3000 2100 50  0001 C CNN
 F 3 "" H 3000 2100 50  0001 C CNN
 	1    3000 2100
@@
 $EndComp
 $Comp
-L GND #PWR101
+L GND #PWR01
 U 1 1 5B1D0556
 P 3350 2550
-F 0 "#PWR101" H 3350 2300 50  0001 C CNN
+F 0 "#PWR01" H 3350 2300 50  0001 C CNN
 F 1 "GND" H 3350 2400 50  0000 C CNN
 F 2 "" H 3350 2550 50  0001 C CNN
@@
 	4800 4650 4500 4650
 $Comp
-L GND #PWR102
+L GND #PWR02
 U 1 1 5B2120C5
 P 7000 6300
-F 0 "#PWR102" H 7000 6050 50  0001 C CNN
+F 0 "#PWR02" H 7000 6050 50  0001 C CNN
 F 1 "GND" H 7000 6150 50  0000 C CNN
 F 2 "" H 7000 6300 50  0001 C CNN

Commit message: Update connector footprints
Parts:
- J101, J103: footprint Pin_Headers:Pin_Header_Angled_1x02_Pitch2.54mm -> Current:Terminal_Block_200_thou
- J102: footprint Pin_Headers:Pin_Header_Angled_1x03_Pitch2.54mm -> Pin_Headers:Pin_Header_Straight_1x03_Pitch2.54mm
Changed lines of the file:
@@
 F 0 "J103" H 7350 2350 50  0000 C CNN
 F 1 "Conn_01x02" V 7450 2200 50  0000 C CNN
-F 2 "Pin_Headers:Pin_Header_Angled_1x02_Pitch2.54mm" H 7350 2250 50  0001 C CNN
+F 2 "Current:Terminal_Block_200_thou" H 7350 2250 50  0001 C CNN
 F 3 "" H 7350 2250 50  0001 C CNN
 	1    7350 2250
@@
 F 0 "J102" H 6050 1950 50  0000 C CNN
 F 1 "Conn_01x03" V 6150 1750 50  0000 C CNN
-F 2 "Pin_Headers:Pin_Header_Angled_1x03_Pitch2.54mm" H 6050 1750 50  0001 C CNN
+F 2 "Pin_Headers:Pin_Header_Straight_1x03_Pitch2.54mm" H 6050 1750 50  0001 C CNN
 F 3 "" H 6050 1750 50  0001 C CNN
 	1    6050 1750
@@
 F 0 "J101" H 3000 2200 50  0000 C CNN
 F 1 "Conn_01x02" V 3100 2050 50  0000 C CNN
-F 2 "Pin_Headers:Pin_Header_Angled_1x02_Pitch2.54mm" H 3000 2100 50  0001 C CNN
+F 2 "Current:Terminal_Block_200_thou" H 3000 2100 50  0001 C CNN
 F 3 "" H 3000 2100 50  0001 C CNN
 	1    3000 2100
