File: PowerRegulation.sch (KiCad schematic (older format))
At the start: 6 parts

Commit message: Initial Annotation
Parts:
- gave numbers to parts that had none: 6
Changed lines of the file:
@@
 $EndDescr
 $Comp
-L GND #PWR?
+L GND #PWR401
 U 1 1 5B20F54A
 P 5800 4000
-F 0 "#PWR?" H 5800 3750 50  0001 C CNN
+F 0 "#PWR401" H 5800 3750 50  0001 C CNN
 F 1 "GND" H 5800 3850 50  0000 C CNN
 F 2 "" H 5800 4000 50  0001 C CNN
@@
 $EndComp
 $Comp
-L C C?
+L C C402
 U 1 1 5B20F550
 P 6600 3550
-F 0 "C?" H 6625 3650 50  0000 L CNN
+F 0 "C402" H 6625 3650 50  0000 L CNN
 F 1 "C" H 6625 3450 50  0000 L CNN
 F 2 "" H 6638 3400 50  0001 C CNN
@@
 $EndComp
 $Comp
-L C C?
+L C C401
 U 1 1 5B20F557
 P 4850 3550
-F 0 "C?" H 4875 3650 50  0000 L CNN
+F 0 "C401" H 4875 3650 50  0000 L CNN
 F 1 "C" H 4875 3450 50  0000 L CNN
 F 2 "" H 4888 3400 50  0001 C CNN
@@
 $EndComp
 $Comp
-L R R?
+L R R403
 U 1 1 5B20F55F
 P 6300 3550
-F 0 "R?" V 6380 3550 50  0000 C CNN
+F 0 "R403" V 6380 3550 50  0000 C CNN
 F 1 "0" V 6300 3550 50  0000 C CNN
 F 2 "" V 6230 3550 50  0001 C CNN
@@
 2.7V
 $Comp
-L LM2931D-R U?
+L LM2931D-R U401
 U 1 1 5B20F567
 P 5850 3600
-F 0 "U?" H 6050 3550 50  0000 C CNN
+F 0 "U401" H 5600 3550 50  0000 C CNN
 F 1 "LM2931D-R" H 5650 4250 50  0000 L CNN
 F 2 "TO_SOT_Packages_THT:TO-220_Vertical" H 5800 4450 50  0001 C CIN
@@
 $EndComp
 $Comp
-L R R?
+L R R401
 U 1 1 5B20F56F
 P 5250 3300
-F 0 "R?" V 5330 3300 50  0000 C CNN
+F 0 "R401" V 5330 3300 50  0000 C CNN
 F 1 "27K" V 5250 3300 50  0000 C CNN
 F 2 "" V 5180 3300 50  0001 C CNN
@@
 $EndComp
 $Comp
-L R R?
+L R R402
 U 1 1 5B20F576
 P 5250 3750
-F 0 "R?" V 5330 3750 50  0000 C CNN
+F 0 "R402" V 5330 3750 50  0000 C CNN
 F 1 "21.6" V 5250 3750 50  0000 C CNN
 F 2 "" V 5180 3750 50  0001 C CNN

Commit message: Added footprints. Created initial netlist.
Parts:
- C401, C402: footprint (none) -> Capacitors_SMD:C_0805_HandSoldering
- R401, R402, R403: footprint (none) -> Resistors_SMD:R_0805
- U401: footprint TO_SOT_Packages_THT:TO-220_Vertical -> SMD_Packages:SOIC-8-N
Changed lines of the file:
@@
 $EndDescr
 $Comp
-L GND #PWR401
+L GND #PWR07
 U 1 1 5B20F54A
 P 5800 4000
-F 0 "#PWR401" H 5800 3750 50  0001 C CNN
+F 0 "#PWR07" H 5800 3750 50  0001 C CNN
 F 1 "GND" H 5800 3850 50  0000 C CNN
 F 2 "" H 5800 4000 50  0001 C CNN
@@
 F 0 "C402" H 6625 3650 50  0000 L CNN
 F 1 "C" H 6625 3450 50  0000 L CNN
-F 2 "" H 6638 3400 50  0001 C CNN
+F 2 "Capacitors_SMD:C_0805_HandSoldering" H 6638 3400 50  0001 C CNN
 F 3 "" H 6600 3550 50  0001 C CNN
 	1    6600 3550
@@
 F 0 "C401" H 4875 3650 50  0000 L CNN
 F 1 "C" H 4875 3450 50  0000 L CNN
-F 2 "" H 4888 3400 50  0001 C CNN
+F 2 "Capacitors_SMD:C_0805_HandSoldering" H 4888 3400 50  0001 C CNN
 F 3 "" H 4850 3550 50  0001 C CNN
 	1    4850 3550
@@
 F 0 "R403" V 6380 3550 50  0000 C CNN
 F 1 "0" V 6300 3550 50  0000 C CNN
-F 2 "" V 6230 3550 50  0001 C CNN
+F 2 "Resistors_SMD:R_0805" V 6230 3550 50  0001 C CNN
 F 3 "" H 6300 3550 50  0001 C CNN
 F 4 "Value" H 6300 3550 60  0001 C CNN "MPN"
@@
 F 0 "U401" H 5600 3550 50  0000 C CNN
 F 1 "LM2931D-R" H 5650 4250 50  0000 L CNN
-F 2 "TO_SOT_Packages_THT:TO-220_Vertical" H 5800 4450 50  0001 C CIN
+F 2 "SMD_Packages:SOIC-8-N" H 5800 4450 50  0001 C CIN
 F 3 "" H 5600 3750 50  0001 C CNN
 	1    5850 3600
@@
 F 0 "R401" V 5330 3300 50  0000 C CNN
 F 1 "27K" V 5250 3300 50  0000 C CNN
-F 2 "" V 5180 3300 50  0001 C CNN
+F 2 "Resistors_SMD:R_0805" V 5180 3300 50  0001 C CNN
 F 3 "" H 5250 3300 50  0001 C CNN
 F 4 "Value" H 5250 3300 60  0001 C CNN "MPN"
@@
 F 0 "R402" V 5330 3750 50  0000 C CNN
 F 1 "21.6" V 5250 3750 50  0000 C CNN
-F 2 "" V 5180 3750 50  0001 C CNN
+F 2 "Resistors_SMD:R_0805" V 5180 3750 50  0001 C CNN
 F 3 "" H 5250 3750 50  0001 C CNN
 	1    5250 3750
