File: $CurrentControl.sch (KiCad schematic (older format))
At the start: 7 parts, among them P1 CONN_01X01, Q401 BUK9575, U201 LMV358

Commit message: Downloaded Chris' files after CSOS Layout session 1 and this is after Session 2.
Moved pots/terms and routed traces to all components.
Parts:
- added C401: C, SMD_Packages:SMD-0805, symbol C
- R401, R402, R403: symbol R-RESCUE-CurrentSinkOrSwim -> R
- RV401: symbol POT-RESCUE-CurrentSinkOrSwim -> POT
- U201: symbol LMV358-RESCUE-CurrentSinkOrSwim -> LMV358
Connections:
- wire segments 22 -> 24
Changed lines of the file:
@@
 EESchema Schematic File Version 2
-LIBS:CurrentSinkOrSwim-rescue
 LIBS:power
 LIBS:device
@@
 LIBS:memory
 LIBS:xilinx
+LIBS:special
 LIBS:microcontrollers
 LIBS:dsp
@@
 $EndDescr
 $Comp
-L LMV358-RESCUE-CurrentSinkOrSwim U201
+L LMV358 U201
 U 2 1 54DADC5E
 P 5500 3700
@@
 $EndComp
 $Comp
-L R-RESCUE-CurrentSinkOrSwim R403
+L R R403
 U 1 1 54DADC66
 P 8100 5150
@@
 Connection ~ 8100 5450
 $Comp
-L POT-RESCUE-CurrentSinkOrSwim RV401
+L POT RV401
 U 1 1 54DADC9B
 P 3750 4050
@@
 	5400 2600 5400 3300
 Connection ~ 3750 2600
+$Comp
+L GND #PWR07
+U 1 1 54DADCA8
+P 4800 3300
+F 0 "#PWR07" H 4800 3050 60  0001 C CNN
+F 1 "GND" H 4800 3150 60  0000 C CNN
+F 2 "" H 4800 3300 60  0000 C CNN
+F 3 "" H 4800 3300 60  0000 C CNN
+	1    4800 3300
+	1    0    0    -1
+$EndComp
+$Comp
+L C C401
+U 1 1 54DADCAE
+P 4800 3050
+F 0 "C401" H 4850 3150 50  0000 L CNN
+F 1 "C" H 4850 2950 50  0000 L CNN
+F 2 "SMD_Packages:SMD-0805" H 4838 2900 30  0001 C CNN
+F 3 "" H 4800 3050 60  0000 C CNN
+	1    4800 3050
+	1    0    0    -1
+$EndComp
+Wire Wire Line
+	4800 2850 4800 2600
+Connection ~ 4800 2600
+Wire Wire Line
+	4800 3300 4800 3250
 Wire Wire Line
 	8100 1500 8100 3500
@@
 	8650 1500 8100 1500
 $Comp
-L R-RESCUE-CurrentSinkOrSwim R402
+L R R402
 U 1 1 54DAE31B
 P 6450 3700
@@
 $EndComp
 $Comp
-L R-RESCUE-CurrentSinkOrSwim R401
+L R R401
 U 1 1 54DADC7B
 P 3750 3100
